Commit message: added table from arena to urdf

File: ur_atc_robot_cell/ur_atc_robot_cell_description/urdf/my_robot_cell.urdf.xacro (robot description, xacro)
@@ -17,5 +17,5 @@
     visual_parameters_file="$(arg visual_parameters_file)"
     >
-      <origin xyz="0 0 1" rpy="0 0 0" />
+      <origin xyz="0 0 0.84" rpy="0 0 0" />
   </xacro:my_robot_cell>
 </robot>

File: ur_atc_robot_cell/ur_atc_robot_cell_description/urdf/my_robot_cell_macro.xacro (robot description, xacro)
@@ -19,57 +19,23 @@
       <visual>
         <geometry>
-          <mesh filename="package://ur_atc_robot_cell_description/meshes/fzi_table.dae"/>
+          <mesh filename="package://ur_atc_robot_cell_description/meshes/table.dae"/>
         </geometry>
-        <origin rpy="0 0 0" xyz="0.75 0.5 -1"/>
+        <origin rpy="0 0 0" xyz="0.75 0.775 -0.84"/>
       </visual>
       <collision>
         <geometry>
-          <mesh filename="package://ur_atc_robot_cell_description/meshes/fzi_table.dae"/>
+          <mesh filename="package://ur_atc_robot_cell_description/meshes/table.dae"/>
         </geometry>
-        <origin rpy="0 0 0" xyz="0.75 0.5 -1"/>
+        <origin rpy="0 0 0" xyz="0.75 0.775 -0.84"/>
       </collision>
     </link>
-    <link name="monitor">
-      <visual>
-        <geometry>
-          <mesh filename="package://ur_atc_robot_cell_description/meshes/171005_Motek_Monitor_L.dae"/>
-        </geometry>
-      </visual>
-      <collision>
-        <geometry>
-          <mesh filename="package://ur_atc_robot_cell_description/meshes/171005_Motek_Monitor_L.dae"/>
-        </geometry>
-      </collision>
-    </link>
-    <joint name="base_to_monitor" type="fixed">
-      <parent link="table"/>
-      <child link="monitor"/>
-      <origin xyz="0.2 0.6 0"/>
-    </joint>
     <material name="white">
       <color rgba="1 1 1 1"/>
     </material>
-    <link name="wall">
-      <visual>
-        <geometry>
-          <mesh filename="package://ur_atc_robot_cell_description/meshes/wall.dae"/>
-        </geometry>
-      </visual>
-      <collision>
-        <geometry>
-          <box size="4.44 0.1 2.5"/>
-        </geometry>
-      </collision>
-    </link>
-    <joint name="base_to_wall" type="fixed">
-      <parent link="table"/>
-      <child link="wall"/>
-      <origin xyz="1.25 1.5 0.5"/>
-    </joint>
     <link name="robot_mount"/>
     <joint name="base_to_robot_mount" type="fixed">
       <parent link="table"/>
       <child link="robot_mount"/>
-      <origin xyz="0.845 0.85 0" rpy="0 0 ${pi}" />
+      <origin xyz="0.58 1.25 0" rpy="0 0 ${pi}" />
     </joint>
     <!--This will create the specific robot-->
