Commit message: branch ur3e_sim

File: ur_atc_robot_cell/ur_atc_robot_cell_description/urdf/my_robot_cell_macro.xacro (robot description, xacro)
@@ -71,5 +71,5 @@
       <parent link="table"/>
       <child link="robot_mount"/>
-      <origin xyz="0.845 0.85 0" rpy="0 0 ${pi}" />
+      <origin xyz="0.845 1.0 0" rpy="0 0 ${pi}" />
     </joint>
     <!--This will create the specific robot-->

Commit message: added tool rack and gripper with tool changer (gripper side) parts to urdf

File: ur_atc_robot_cell/ur_atc_robot_cell_description/urdf/my_robot_cell_macro.xacro (robot description, xacro)
@@ -2,4 +2,6 @@
 <robot xmlns:xacro="http://ros.org/wiki/xacro">
   <xacro:include filename="$(find ur_description)/urdf/ur_macro.xacro"/>
+  <xacro:include filename="$(find ur_atc_robot_cell_description)/urdf/tool_rack.xacro"/>
+  <xacro:include filename="$(find ur_atc_robot_cell_description)/urdf/gripper_side_TC.xacro" />
   <xacro:macro name="my_robot_cell" params="
     parent
@@ -51,4 +53,14 @@
       <origin xyz="0 0 0" rpy="0 0 0" />
     </xacro:ur_robot>
+    <xacro:property name="tool_rack_x_dist" value="0.77" />
+    <xacro:property name="tool_rack_y_dist" value="0.23" />
+    <link name="tool_rack_base"/>
+    <joint name="tool_rack_base" type="fixed">
+      <parent link="table" />
+      <child link="tool_rack_base" />
+      <origin xyz="${tool_rack_x_dist} ${tool_rack_y_dist} 0" rpy="0 0 0" />
+    </joint>
+    <xacro:tool-rack parent="tool_rack_base"/>
+    <xacro:gripper-tool-change-adaptor parent_link="ratelier_link"/>
   </xacro:macro>
 </robot>
