Commit message: added mesh files for the gripper, modified xacro to find the right package

File: ur_atc_robot_cell/ur_atc_robot_cell_description/urdf/gripper_side_TC.xacro (robot description, xacro)
@@ -15,5 +15,5 @@
             <origin xyz="0 -0.0109987 0.0115755" rpy="1.5708 0 1.5708"/>
             <geometry>
-                <mesh filename="package://igus_robot_cell/meshes/iso_50_flange_schunk_v1.stl"/>
+                <mesh filename="package://ur_atc_robot_cell_description/meshes/iso_50_flange_schunk_v1.stl"/>
             </geometry>
             <material name="iso_50_flange_schunk_v1_material">
@@ -24,5 +24,5 @@
             <origin xyz="0 -0.0109987 0.0115755" rpy="1.5708 0 1.5708"/>
             <geometry>
-                <mesh filename="package://igus_robot_cell/meshes/iso_50_flange_schunk_v1.stl"/>
+                <mesh filename="package://ur_atc_robot_cell_description/meshes/iso_50_flange_schunk_v1.stl"/>
             </geometry>
             </collision>
@@ -31,5 +31,5 @@
             <origin xyz="0 -0.0109987 -0.0104245" rpy="-1.5708 -0 0"/>
             <geometry>
-                <mesh filename="package://igus_robot_cell/meshes/base_link_gripper_base.stl"/>
+                <mesh filename="package://ur_atc_robot_cell_description/meshes/base_link_gripper_base.stl"/>
             </geometry>
             <material name="base_link_gripper_base_material">
@@ -40,5 +40,5 @@
             <origin xyz="0 -0.0109987 -0.0104245" rpy="-1.5708 -0 0"/>
             <geometry>
-                <mesh filename="package://igus_robot_cell/meshes/base_link_gripper_base.stl"/>
+                <mesh filename="package://ur_atc_robot_cell_description/meshes/base_link_gripper_base.stl"/>
             </geometry>
             </collision>
@@ -47,5 +47,5 @@
             <origin xyz="-0.00125 -0.0109987 0.0360255" rpy="-0 0 -0"/>
             <geometry>
-                <mesh filename="package://igus_robot_cell/meshes/adaptor_parts.stl"/>
+                <mesh filename="package://ur_atc_robot_cell_description/meshes/adaptor_parts.stl"/>
             </geometry>
             <material name="adaptor_parts_material">
@@ -56,5 +56,5 @@
             <origin xyz="-0.00125 -0.0109987 0.0360255" rpy="-0 0 -0"/>
             <geometry>
-                <mesh filename="package://igus_robot_cell/meshes/adaptor_parts.stl"/>
+                <mesh filename="package://ur_atc_robot_cell_description/meshes/adaptor_parts.stl"/>
             </geometry>
             </collision>
@@ -63,5 +63,5 @@
             <origin xyz="-0.00125 -0.0109987 0.0115755" rpy="-0 0 1.5708"/>
             <geometry>
-                <mesh filename="package://igus_robot_cell/meshes/adaptor_parts__2.stl"/>
+                <mesh filename="package://ur_atc_robot_cell_description/meshes/adaptor_parts__2.stl"/>
             </geometry>
             <material name="adaptor_parts_2_material">
@@ -72,5 +72,5 @@
             <origin xyz="-0.00125 -0.0109987 0.0115755" rpy="-0 0 1.5708"/>
             <geometry>
-                <mesh filename="package://igus_robot_cell/meshes/adaptor_parts__2.stl"/>
+                <mesh filename="package://ur_atc_robot_cell_description/meshes/adaptor_parts__2.stl"/>
             </geometry>
             </collision>
@@ -79,5 +79,5 @@
             <origin xyz="-0.00125 -0.0109987 0.0298255" rpy="-3.14159 0 1.5708"/>
             <geometry>
-                <mesh filename="package://igus_robot_cell/meshes/adaptor_parts__3.stl"/>
+                <mesh filename="package://ur_atc_robot_cell_description/meshes/adaptor_parts__3.stl"/>
             </geometry>
             <material name="adaptor_parts_3_material">
@@ -88,5 +88,5 @@
             <origin xyz="-0.00125 -0.0109987 0.0298255" rpy="-3.14159 0 1.5708"/>
             <geometry>
-                <mesh filename="package://igus_robot_cell/meshes/adaptor_parts__3.stl"/>
+                <mesh filename="package://ur_atc_robot_cell_description/meshes/adaptor_parts__3.stl"/>
             </geometry>
             </collision>
@@ -95,5 +95,5 @@
             <origin xyz="-0.00125 -0.0109987 0.0318255" rpy="-3.14159 0 1.5708"/>
             <geometry>
-                <mesh filename="package://igus_robot_cell/meshes/adaptor_parts__4.stl"/>
+                <mesh filename="package://ur_atc_robot_cell_description/meshes/adaptor_parts__4.stl"/>
             </geometry>
             <material name="adaptor_parts_4_material">
@@ -104,5 +104,5 @@
             <origin xyz="-0.00125 -0.0109987 0.0318255" rpy="-3.14159 0 1.5708"/>
             <geometry>
-                <mesh filename="package://igus_robot_cell/meshes/adaptor_parts__4.stl"/>
+                <mesh filename="package://ur_atc_robot_cell_description/meshes/adaptor_parts__4.stl"/>
             </geometry>
             </collision>
@@ -111,5 +111,5 @@
             <origin xyz="-0.00125 -0.0109987 0.0522255" rpy="3.14159 -0 -1.5708"/>
             <geometry>
-                <mesh filename="package://igus_robot_cell/meshes/base_link.stl"/>
+                <mesh filename="package://ur_atc_robot_cell_description/meshes/base_link.stl"/>
             </geometry>
             <material name="base_link_material">
@@ -120,5 +120,5 @@
             <origin xyz="-0.00125 -0.0109987 0.0522255" rpy="3.14159 -0 -1.5708"/>
             <geometry>
-                <mesh filename="package://igus_robot_cell/meshes/base_link.stl"/>
+                <mesh filename="package://ur_atc_robot_cell_description/meshes/base_link.stl"/>
             </geometry>
             </collision>
@@ -127,5 +127,5 @@
             <origin xyz="-0.00525 0.0112012 0.0115755" rpy="-0 -0 -1.5708"/>
             <geometry>
-                <mesh filename="package://igus_robot_cell/meshes/adaptor_parts__5.stl"/>
+                <mesh filename="package://ur_atc_robot_cell_description/meshes/adaptor_parts__5.stl"/>
             </geometry>
             <material name="adaptor_parts_5_material">
@@ -136,5 +136,5 @@
             <origin xyz="-0.00525 0.0112012 0.0115755" rpy="-0 -0 -1.5708"/>
             <geometry>
-                <mesh filename="package://igus_robot_cell/meshes/adaptor_parts__5.stl"/>
+                <mesh filename="package://ur_atc_robot_cell_description/meshes/adaptor_parts__5.stl"/>
             </geometry>
             </collision>
@@ -151,5 +151,5 @@
             <origin xyz="0.02615 -0.0096 0.027" rpy="-1.5708 -1.5708 0"/>
             <geometry>
-                <mesh filename="package://igus_robot_cell/meshes/schunk_5522661_finger_egp_64.stl"/>
+                <mesh filename="package://ur_atc_robot_cell_description/meshes/schunk_5522661_finger_egp_64.stl"/>
             </geometry>
             <material name="schunk_5522661_finger_egp_64_material">
@@ -160,5 +160,5 @@
             <origin xyz="0.02615 -0.0096 0.027" rpy="-1.5708 -1.5708 0"/>
             <geometry>
-                <mesh filename="package://igus_robot_cell/meshes/schunk_5522661_finger_egp_64.stl"/>
+                <mesh filename="package://ur_atc_robot_cell_description/meshes/schunk_5522661_finger_egp_64.stl"/>
             </geometry>
             </collision>
@@ -167,5 +167,5 @@
             <origin xyz="0.02615 -0.0096 0.027" rpy="-1.5708 -1.5708 0"/>
             <geometry>
-                <mesh filename="package://igus_robot_cell/meshes/finger.stl"/>
+                <mesh filename="package://ur_atc_robot_cell_description/meshes/finger.stl"/>
             </geometry>
             <material name="finger_material">
@@ -176,5 +176,5 @@
             <origin xyz="0.02615 -0.0096 0.027" rpy="-1.5708 -1.5708 0"/>
             <geometry>
-                <mesh filename="package://igus_robot_cell/meshes/finger.stl"/>
+                <mesh filename="package://ur_atc_robot_cell_description/meshes/finger.stl"/>
             </geometry>
             </collision>
@@ -199,5 +199,5 @@
             <origin xyz="-0.02615 0.0096 0.027" rpy="1.5708 -1.5708 0"/>
             <geometry>
-                <mesh filename="package://igus_robot_cell/meshes/schunk_5522661_finger_egp_64.stl"/>
+                <mesh filename="package://ur_atc_robot_cell_description/meshes/schunk_5522661_finger_egp_64.stl"/>
             </geometry>
             <material name="schunk_5522661_finger_egp_64_2_material">
@@ -208,5 +208,5 @@
             <origin xyz="-0.02615 0.0096 0.027" rpy="1.5708 -1.5708 0"/>
             <geometry>
-                <mesh filename="package://igus_robot_cell/meshes/schunk_5522661_finger_egp_64.stl"/>
+                <mesh filename="package://ur_atc_robot_cell_description/meshes/schunk_5522661_finger_egp_64.stl"/>
             </geometry>
             </collision>
@@ -215,5 +215,5 @@
             <origin xyz="-0.02615 0.0096 0.027" rpy="1.5708 -1.5708 0"/>
             <geometry>
-                <mesh filename="package://igus_robot_cell/meshes/finger.stl"/>
+                <mesh filename="package://ur_atc_robot_cell_description/meshes/finger.stl"/>
             </geometry>
             <material name="finger_2_material">
@@ -224,5 +224,5 @@
             <origin xyz="-0.02615 0.0096 0.027" rpy="1.5708 -1.5708 0"/>
             <geometry>
-                <mesh filename="package://igus_robot_cell/meshes/finger.stl"/>
+                <mesh filename="package://ur_atc_robot_cell_description/meshes/finger.stl"/>
             </geometry>
             </collision>
